Commit message: mercury_ros -> reorientbot_ros

File: reorientbot/_pybullet/data/franka_panda/panda_drl.urdf (robot description, URDF)
Before this commit: robot panda, 11 links, 10 joints
Links:
- link panda_suction_gripper: geometry collision mesh filename=package://reorientbot_ros/robots/drl/meshes/collision/sucti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; visual mesh filename=package://reorientbot_ros/robots/drl/meshes/visual/suction_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

File: reorientbot/_pybullet/data/franka_panda/panda_drl.urdf.xacro (robot description, xacro)
@@ -2,5 +2,5 @@
 <robot xmlns:xacro="http://www.ros.org/wiki/xacro" name="panda">
   <xacro:include filename="panda_arm.urdf"/>
-  <xacro:include filename="$(find mercury_ros)/robots/drl/suction.xacro"/>
+  <xacro:include filename="$(find reorientbot_ros)/robots/drl/suction.xacro"/>
   <xacro:suction_gripper ns="panda" rpy="${pi} 0 ${-pi/4}" xyz="0 0 0.0065" connected_to="panda_link8"/>
 </robot>

File: ros/src/reorientbot_ros/robots/drl/suction.xacro (robot description, xacro)
@@ -18,5 +18,5 @@
       <visual>
         <geometry>
-          <mesh filename="package://mercury_ros/robots/drl/meshes/visual/suction_mount.obj"/>
+          <mesh filename="package://reorientbot_ros/robots/drl/meshes/visual/suction_mount.obj"/>
         </geometry>
         <material name="black"/>
@@ -24,5 +24,5 @@
       <collision>
         <geometry>
-          <mesh filename="package://mercury_ros/robots/drl/meshes/collision/suction_mount.obj"/>
+          <mesh filename="package://reorientbot_ros/robots/drl/meshes/collision/suction_mount.obj"/>
         </geometry>
       </collision>

File: ros/src/reorientbot_ros/robots/panda_drl.urdf.xacro (robot description, xacro)
@@ -2,5 +2,5 @@
 <robot xmlns:xacro="http://www.ros.org/wiki/xacro" name="panda">
   <xacro:include filename="$(find franka_description)/robots/panda_arm.urdf.xacro"/>
-  <xacro:include filename="$(find mercury_ros)/robots/drl/suction.xacro"/>
+  <xacro:include filename="$(find reorientbot_ros)/robots/drl/suction.xacro"/>
   <xacro:suction_gripper ns="panda" rpy="${pi} 0 ${-pi/4}" xyz="0 0 0.0065" connected_to="panda_link8"/>
 </robot>
